File: schematics/kiCad/blinky-cube.kicad_pcb (KiCad board)
At the start: 2 copper layers, 86.4 x 48.3 mm, 17 parts, among them J1 901-9894-RFX, J2 Barrel_Jack_Switch, SW1 SW_Push, U1 Pico, U2 LM4040LP-3

Commit message: added logo
Parts:
- added G***: LOGO, blinkyLiteLogo:blinkyLiteLogo, F.Cu at (119.4, 113.7)
Other:
- board text added: "blinky-rf-power-meter-v1"
